File: src/kicad-solo/Megatone-solo.sch (KiCad schematic (older format))
At the start: 21 parts, among them P1 CONN_01X01, P2 CONN_01X01, SW1 LORLIN_1X12

Commit message: 2014-10-21--2
Parts:
- C1: renamed from C9; footprint (none) -> libcms:SM0805
- C2: renamed from C8; footprint (none) -> libcms:SM0805
- C3: renamed from C7; footprint (none) -> libcms:SM0805
- C4: renamed from C6; footprint (none) -> libcms:SM0805
- C5, R5: footprint (none) -> libcms:SM0805
- C6: renamed from C4; value 4700 p -> 4700p; footprint (none) -> libcms:SM0805
- C7: renamed from C3; value 2200 p -> 2200p; footprint (none) -> libcms:SM0805
- C8: renamed from C2; value 1000 p -> 1000p; footprint (none) -> libcms:SM0805
- C9: renamed from C1; value 470 p -> 470p; footprint (none) -> libcms:SM0805
- P1, P2: footprint (none) -> Pin_Headers:Pin_Header_Straight_1x01
- R1: renamed from R9; footprint (none) -> libcms:SM0805
- R2: renamed from R8; footprint (none) -> libcms:SM0805
- R3: renamed from R7; footprint (none) -> libcms:SM0805
- R4: renamed from R6; footprint (none) -> libcms:SM0805
- R6: renamed from R4; footprint (none) -> libcms:SM0805
- R7: renamed from R3; footprint (none) -> libcms:SM0805
- R8: renamed from R2; footprint (none) -> libcms:SM0805
- R9: renamed from R1; footprint (none) -> libcms:SM0805
- SW1: footprint (none) -> Custom:Lorlin_CK_1p12t
Other:
- moved on the sheet: C1, C2, C3, C4, C5, C6, C7, C8, C9, P1, P2, R1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
