File: src/kicad-solo/Megatone-solo.kicad_pcb (KiCad board)
At the start: 2 copper layers, 27.4 x 27.4 mm, 21 parts, among them P1 CONN_01X01, P2 CONN_01X01, SW1 LORLIN_1X12

Commit message: 2014-10-23 - updated solo and duo pcbs
Parts:
- moved P2 6.48 mm to (148.6, 97.3)
- moved P1 6.43 mm to (142.2, 99.1)
Connections:
- SW1 pad 10: (no net) -> Net-(SW1-Pad10)
- SW1 pad 11: (no net) -> Net-(SW1-Pad11)
- SW1 pad 12: (no net) -> Net-(SW1-Pad12)
Routing:
- net GND: track 70.3 -> 73.1 mm
Other:
- board size 27.4 x 27.4 mm -> 26.9 x 27.9 mm

Commit message: update pcbs and generate fab plots
Parts:
- turned P1 to 90 degrees
- turned P2 to 30 degrees
Other:
- board text added: "Megatone Solo v5 dolganoff.com/fr/a-propos Open Hardware"
