File: src/kicad-solo/Megatone-solo.kicad_pcb (KiCad board)
At the start: 2 copper layers, 26.9 x 27.9 mm, 21 parts, among them P1 CONN_01X01, P2 CONN_01X01, SW1 LORLIN_1X12

Commit message: moving output pins
Parts:
- moved P2 0.80 mm to (149.4, 97.0)
