File: src/kicad-duo/Megatone-duo.kicad_pcb (KiCad board)
At the start: 2 copper layers, 27.4 x 28.4 mm, 22 parts, among them P1 Classic, P2 Boost, P3 Gnd, SW1 LORLIN_2X6

Commit message: M. Duo: corrected wrong cap values on boost side
Parts:
- C1: value 47n -> 1n
- C2: value 22n -> 2.2n
- C3: value 10n -> 4.7n
- C4: value 4700p -> 10n
- C5: value 2200p -> 22n
- C6: value 1000p -> 47n

Commit message: Revert "M. Duo: corrected wrong cap values on boost side"
This reverts commit b441f0806059993cadffced08bf4fcd550c3232b.
Parts:
- C1: value 1n -> 47n
- C2: value 2.2n -> 22n
- C3: value 4.7n -> 10n
- C4: value 10n -> 4700p
- C5: value 22n -> 2200p
- C6: value 47n -> 1000p
